File: pic-gym/_saved_pic-gym.sch (KiCad schematic (older format))
At the start: 30 parts, among them CON1 BARREL_JACK, SW1 SW_SPST, SW2 SW_Push, SW3 SW_DIP_x05, U1 LM7805, U2 PIC16F84A-XX/P, Y1 4MHz

Commit message: 3D correct
Parts:
- U1: footprint TO_SOT_Packages_THT:TO-220_Neutral123_Vertical_LargePads -> TO_SOT_Packages_THT:TO-220_Neutral123_Vertical
Changed lines of the file:
@@
-$EndComp
-$Comp
-L LM7805 U1
-U 1 1 58853EA6
-P 4600 6400
-F 0 "U1" H 4750 6204 50  0000 C CNN
-F 1 "LM7805" H 4600 6600 50  0000 C CNN
-F 2 "TO_SOT_Packages_THT:TO-220_Neutral123_Vertical_LargePads" H 4600 6400 50  0001 C CNN
-F 3 "" H 4600 6400 50  0001 C CNN
-	1    4600 6400
-	1    0    0    -1
 $EndComp
 $Comp
@@
 	0    1    1    0
 $EndComp
+$Comp
+L LM7805 U1
+U 1 1 5887B1EF
+P 4600 6400
+F 0 "U1" H 4750 6204 50  0000 C CNN
+F 1 "LM7805" H 4600 6600 50  0000 C CNN
+F 2 "TO_SOT_Packages_THT:TO-220_Neutral123_Vertical" H 4600 6400 50  0001 C CNN
+F 3 "" H 4600 6400 50  0001 C CNN
+	1    4600 6400
+	1    0    0    -1
+$EndComp
 $EndSCHEMATC
