File: pic-gym/pic-gym.kicad_pcb (KiCad board)
At the start: 2 copper layers, 63.5 x 55 mm, 30 parts, among them CON1 BARREL_JACK, SW1 SW_SPST, SW2 SW_Push, SW3 SW_DIP_x05, U1 LM7805, U2 PIC16F84A-XX/P, Y1 4MHz

Commit message: Improving schematic
Connections:
- CON1 pad 1: GND -> Net-(CON1-Pad1)
- CON1 pad 2: Net-(CON1-Pad2) -> GND
- SW1 pad 1: Net-(CON1-Pad2) -> Net-(CON1-Pad1)
Routing:
- net Net-(CON1-Pad2): track 16.7 -> 0.00 mm
- net Net-(CON1-Pad1): track 0.00 -> 8.71 mm
- net GND: track 134.9 -> 135.7 mm
