File: pic-gym/pic-gym.sch (KiCad schematic (older format))
At the start: 30 parts, among them CON1 BARREL_JACK, SW1 SW_SPST, SW2 SW_Push, SW3 SW_DIP_x05, U1 LM7805, U2 PIC16F84A-XX/P, Y1 4MHz

Commit message: Improving schematic
Parts:
- U1: symbol LM7805 -> LM7805-RESCUE-pic-gym
Connections:
- net +5V: now also U1.3 (VO); no longer U1.VO
- net GND: now also CON1.2, U1.2 (GND); no longer CON1.1, U1.GND
- net at SW1.1 (A): now also CON1.1; no longer CON1.2
- net at C3.1, C4.1, D1.1 (K): now also U1.1 (VI); no longer U1.VI
Changed lines of the file:
@@
 EESchema Schematic File Version 2
+LIBS:pic-gym-rescue
 LIBS:power
 LIBS:device
@@
 Wire Wire Line
 	6850 1000 7100 1000
-Wire Wire Line
-	2150 6350 2550 6350
 $Comp
 L GND #PWR010
@@
 	1    0    0    -1
 $EndComp
-Wire Wire Line
-	2150 6150 2250 6150
-Wire Wire Line
-	2250 6150 2250 6900
 Wire Wire Line
 	3550 6800 3550 6900
@@
 $EndComp
 $Comp
-L LM7805 U1
+L LM7805-RESCUE-pic-gym U1
 U 1 1 5887B1EF
 P 4600 6400
@@
 	1    0    0    -1
 $EndComp
+Wire Wire Line
+	2150 6150 2500 6150
+Wire Wire Line
+	2500 6150 2500 6350
+Wire Wire Line
+	2500 6350 2550 6350
+Wire Wire Line
+	2250 6900 2250 6350
+Wire Wire Line
+	2250 6350 2150 6350
 $EndSCHEMATC
